Commit message: new arm file

File: final_project/controllers/grocery_shopper/arm.urdf (robot description, URDF)
Before this commit: robot TIAGo Steel, 13 links, 12 joints
Links:
- added link gripper_right_finger_link; collision box size=0.0055 0.0295 0.018; collision box size=0.0076 0.05091 0.08982
Joints:
- added joint gripper_right_finger_joint: type prismatic, parent front, child gripper_right_finger_link, origin xyz=0 0 0 rpy=0 0 0, axis 1 0 0, limit lower=0 upper=0.045 effort=16 velocity=0.05

Commit message: rrt*

File: final_project/controllers/grocery_shopper/arm.urdf (robot description, URDF)
Before this commit: robot TIAGo Steel, 14 links, 13 joints
Links:
- removed link gripper_right_finger_link
Joints:
- removed joint gripper_right_finger_joint
